File: Electronic-design/Stage-by-stage-design/01_Digital-interface/KiCad_files/Digital_Interface/Digital_Interface.kicad_sch (KiCad schematic)
At the start: 33 parts, among them J1 Keyboard_3x4, J10 Conn_01x06_Pin, J2 LCD_SCREEN, J3 DAC1, J4 DAC2, J5 ADC1, J6 ADC2, J7 DAC1, J8 DAC2, J9 3.3V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

Commit message: Added test digital interface PCB
Parts:
- C1, C2, C3, C4, C5: footprint (none) -> Capacitor_THT:C_Disc_D5.0mm_W2.5mm_P5.00mm
- D1, D2, D3: footprint (none) -> LED_THT:LED_D5.0mm
- J1: footprint (none) -> Connector_PinHeader_2.54mm:PinHeader_1x07_P2.54mm_Vertical
- J10: footprint (none) -> Connector_PinHeader_2.54mm:PinHeader_1x06_P2.54mm_Vertical
- J2: footprint (none) -> Connector_PinHeader_2.54mm:PinHeader_1x04_P2.54mm_Vertical
- J3, J4: footprint (none) -> Library:MCP4725_module
- J5, J6, J7, J8, J9: footprint (none) -> Connector_PinHeader_2.54mm:PinHeader_1x02_P2.54mm_Vertical
- R1, R10, R11, R2, R3, R4, R5, R6, R7, R8, R9: footprint (none) -> Resistor_THT:R_Axial_DIN0207_L6.3mm_D2.5mm_P7.62mm_Horizontal
- SW1, SW2, SW3: footprint (none) -> Button_Switch_THT:SW_PUSH_6mm
- U2: footprint SOIC28_SO_MCH -> Library:SOIC28_SO_MCH
Connections:
- net at J1.4 (Pin_4): now also U2.18 (RC7); no longer U2.13 (RC2)
- net at J1.5 (Pin_5): now also U2.17 (RC6); no longer U2.16 (RC5)
- net at J1.6 (Pin_6): now also U2.16 (RC5); no longer U2.17 (RC6)
- net at J1.7 (Pin_7): now also U2.13 (RC2); no longer U2.18 (RC7)
