File: Electronic-design/General-Design/PCB/02_Power-supply/PCB60hz_15/PCB60hz_15.kicad_pcb (KiCad board)
At the start: 2 copper layers, 91 x 48 mm, 27 parts, among them IC1 TPS54302DDCR, IC2 L7812CV, IC3 L7912CV, J1 4300.0104, J2 -12V, J3 +12V, J4 +5V, T1 3FS-324

Commit message: PCB60HZ-Fix
Parts:
- added ?: , , F.Cu at (113.7, 88.8)
- added REF**: GND_MH, MountingHole:GND_MountingHole, F.Cu at (106.1, 92.5)
- moved C5 1.92 mm to (113.8, 86.0)
- moved C2 0.30 mm to (98.2, 97.5)
Connections:
- C2 pad 1: Net-(D2-A) -> GNDREF
- C2 pad 2: GNDREF -> Net-(D2-A)
Routing:
- net Net-(T1-PRI_2): track 22.4 -> 10.5 mm
- net Net-(T1-PRI_1): track 19.5 -> 9.16 mm
- net Net-(D3-K): track 65.2 -> 69.6 mm, vias 1 -> 0
- net Net-(IC1-BOOT): track 3.47 -> 7.03 mm
- net Net-(D2-A): track 54.9 -> 51.4 mm
- net Net-(IC1-SW): track 20.8 -> 22.3 mm
- net GNDREF: vias 3 -> 0
Other:
- board text added: "Prototipo #2 Fuente AC->DC +5V y ±12V"
- board text removed: "Prototipo #1 Fuente AC->DC +5V y ±12V"
