File: Electronic-design/General-Design/PCB/02_Power-supply/PCB60hz_15/PCB60hz_15.kicad_sch (KiCad schematic)
At the start: 27 parts, among them IC1 TPS54302DDCR, IC2 L7812CV, IC3 L7912CV, J1 4300.0104, J2 -12V, J3 +12V, J4 +5V, T1 3FS-324

Commit message: PCB60HZ-Fix
Connections:
- net GNDREF: now also C2.1; no longer C2.2
- net at C9.1, D2.2 (A), D4.2 (A)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: now also C2.2; no longer C2.1
Other:
- moved on the sheet: C2
Changed lines of the file:
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@@
 	(symbol
 		(lib_id "Device:C_Polarized")
-		(at 115.57 86.36 180)
+		(at 115.57 86.36 0)
 		(unit 1)
 		(exclude_from_sim no)
@@
 		(dnp no)
 		(property "Reference" "C2"
-			(at 118.364 88.9 0)
+			(at 112.776 83.82 0)
 			(effects
 				(font
@@
 		)
 		(property "Value" "680uF"
-			(at 117.094 90.932 0)
+			(at 114.046 81.788 0)
 			(effects
 				(font
@@
 		)
 		(property "Footprint" "Capacitor_THT:CP_Radial_D10.0mm_P5.00mm"
-			(at 114.6048 82.55 0)
+			(at 116.5352 90.17 0)
 			(effects
 				(font

Commit message: PSIM-FLYBACK-FINAL
Parts:
- C7, C8: value 100nF -> 220nF
- R1: value 100k -> 100k- Aunque medido da como 90k creo
Changed lines of the file:
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@@
 			)
 		)
-		(property "Value" "100nF"
+		(property "Value" "220nF"
 			(at 135.636 81.788 0)
 			(effects
@@
 			)
 		)
-		(property "Value" "100nF"
+		(property "Value" "220nF"
 			(at 136.398 76.454 0)
 			(effects
@@
 			)
 		)
-		(property "Value" "100k"
+		(property "Value" "100k- Aunque medido da como 90k creo"
 			(at 226.06 105.4099 0)
 			(effects
