File: Electronic-design/General-Design/PCB/03_Power-supply-Flyback/Flyback_PCB_60Hz/Flyback_PCB_60Hz.kicad_sch (KiCad schematic)
At the start: 53 parts, among them IC4 UCC38C43DGKR, J1 4300.0104, J6 Conn_01x02, Q1 NMOS, Q2 PNP, Q3 NPN, T2 Transformer_1P_2S, U1 4N35, U2 TL431LP

Commit message: MOV
Parts:
- added RV1: Varistor, symbol Device:Varistor
Connections:
- net Supplies/N: now also RV1.2; no longer F1.1
- new net: F1.1, RV1.1
Changed lines of the file:
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@@
 	(wire
 		(pts
+			(xy 50.8 48.26) (xy 53.34 48.26)
+		)
+		(stroke
+			(width 0)
+			(type default)
+		)
+	)
+	(wire
+		(pts
 			(xy 168.91 24.13) (xy 168.91 41.91)
 		)
@@
 	(wire
 		(pts
-			(xy 40.64 48.26) (xy 53.34 48.26)
-		)
-		(stroke
-			(width 0)
-			(type default)
-		)
-	)
-	(wire
-		(pts
 			(xy 168.91 111.76) (xy 168.91 110.49)
 		)
@@
 	(wire
 		(pts
+			(xy 40.64 48.26) (xy 43.18 48.26)
+		)
+		(stroke
+			(width 0)
+			(type default)
+		)
+	)
+	(wire
+		(pts
 			(xy 227.33 161.29) (xy 227.33 160.02)
 		)
@@
 					(unit 1)
 				)
+			)
+		)
+	)
+	(symbol
+		(lib_id "Device:Varistor")
+		(at 46.99 48.26 270)
+		(unit 1)
+		(exclude_from_sim no)
+		(in_bom yes)
+		(on_board yes)
+		(dnp no)
+		(fields_autoplaced yes)
+		(property "Reference" "RV1"
+			(at 46.7966 40.64 90)
+			(effects
+				(font
+					(size 1.27 1.27)
+				)
+			)
+		)
+		(property "Value" "Varistor"
+			(at 46.7966 43.18 90)
+			(effects
+				(font
+					(size 1.27 1.27)
+				)
+			)
+		)
+		(property "Footprint" ""
+			(at 46.99 46.482 90)
+			(effects
+				(font
+					(size 1.27 1.27)
+				)
+				(hide yes)
+			)
+		)
+		(property "Datasheet" "~"
+			(at 46.99 48.26 0)
+			(effects
+				(font
+					(size 1.27 1.27)
+				)
+				(hide yes)
+			)
+		)
+		(property "Description" "Voltage dependent resistor"
+			(at 46.99 48.26 0)
+			(effects
+				(font
+					(size 1.27 1.27)
+				)
+				(hide yes)
+			)
+		)
+		(property "Sim.Name" "kicad_builtin_varistor"
+			(at 46.99 48.26 0)
+			(effects
+				(font
+					(size 1.27 1.27)
+				)
+				(hide yes)
+			)
+		)
+		(property "Sim.Device" "SUBCKT"
+			(at 46.99 48.26 0)
+			(effects
+				(font
+					(size 1.27 1.27)
+				)
+				(hide yes)
+			)
+		)
+		(property "Sim.Pins" "1=A 2=B"
+			(at 46.99 48.26 0)
+			(effects
+				(font
+					(size 1.27 1.27)
+				)
+				(hide yes)
+			)
+		)
+		(property "Sim.Params" "threshold=1k"
+			(at 46.99 48.26 0)
+			(effects
+				(font
+					(size 1.27 1.27)
+				)
+				(hide yes)
+			)
+		)
+		(property "Sim.Library" "${KICAD7_SYMBOL_DIR}/Simulation_SPICE.sp"
+			(at 46.99 48.26 0)
+			(effects
+				(font
+					(size 1.27 1.27)
+				)
+				(hide yes)
+			)
+		)
+		(pin "1"
+		)
+		(pin "2"
+		)
+		(instances
+			(project ""
+				(path "/e667b3b5-58bf-48ce-ba71-7e90a3c6a4c9"
+					(reference "RV1")
+					(unit 1)
+				)

Commit message: Wololo-Footprints-Flyback-1
Parts:
- removed IC4: UCC38C43DGKR, Footprints:SOP65P490X110-8N, symbol UCC38C43DGKR:UCC38C43DGKR
- removed U1: 4N35, Package_DIP:DIP-6_W7.62mm, symbol Isolator:4N35
- removed U2: TL431LP, Package_TO_SOT_THT:TO-92_Inline, symbol Reference_Voltage:TL431LP
- added C23: R46KI310050M1K, Flyback:R46KI310050M1K, symbol F_1_R46KI310050M1K:R46KI310050M1K
- added IC4: DPC817L-A-TR, Flyback:SOP254P1180X410-4N, symbol F_1_DPC817L-A-TR:DPC817L-A-TR
- added IC5: UCC38C43DR, Flyback:SOIC127P600X175-8N, symbol F_1_UCC38C43DR:UCC38C43DR
- added IC6: TL431ACLPR, TL431ACLPR, symbol F_1_TL431ACLPR:TL431ACLPR
- added R27: 1k, Resistor_SMD:R_0603_1608Metric_Pad0.98x0.95mm_HandSolder, symbol Device:R_US
- C11: value C -> 1u; footprint (none) -> Capacitor_SMD:C_0805_2012Metric_Pad1.18x1.45mm_HandSolder
- C12: value C -> 7n; footprint (none) -> Capacitor_SMD:C_0805_2012Metric_Pad1.18x1.45mm_HandSolder
- C13: value C -> 1nF; footprint (none) -> Capacitor_SMD:C_0805_2012Metric_Pad1.18x1.45mm_HandSolder
- C14: footprint (none) -> Capacitor_SMD:C_0805_2012Metric_Pad1.18x1.45mm_HandSolder
- C15: value C -> 470pF; footprint (none) -> Capacitor_SMD:C_0805_2012Metric_Pad1.18x1.45mm_HandSolder
- C16: value C_Polarized -> 618uF; footprint (none) -> Capacitor_THT:CP_Radial_D10.0mm_P5.00mm
- C17, C19: value C -> 100nF; footprint (none) -> Capacitor_SMD:C_0805_2012Metric_Pad1.18x1.45mm_HandSolder
- C18: value C -> 22u
- R10, R7: value R_US -> 10k; footprint (none) -> Resistor_SMD:R_0603_1608Metric_Pad0.98x0.95mm_HandSolder
- R11: value R_US -> 4k; footprint (none) -> Resistor_SMD:R_0603_1608Metric_Pad0.98x0.95mm_HandSolder
- R12: value R_US -> 15k; footprint (none) -> Resistor_SMD:R_0603_1608Metric_Pad0.98x0.95mm_HandSolder
- R13: value R_US -> 24k; footprint (none) -> Resistor_SMD:R_0603_1608Metric_Pad0.98x0.95mm_HandSolder
- R14: value R_US -> 1k
- R21: value R_US -> 0.250
- R5: value R_US -> 47k
Connections:
- net GND: now also IC6.2 (A)
- net GNDREF: now also IC5.5 (GND)
- net Supplies/L: now also C23.2
- net Supplies/N: now also C23.1
- net Vref: now also IC5.8 (VREF)
- net at C21.2, R24.2, R25.1: now also IC6.1 (REF)
- net at C14.1, Q2.3 (E), R7.1: now also IC5.1 (COMP)
- net at C14.2, R15.1, R7.2: now also IC5.2 (FB)
- net at C18.1, C19.2, D10.1 (K)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: now also IC5.7 (VDD)
- net at C15.1, R17.1, R26.1: now also IC5.3 (CS), R27.2; no longer R13.2
- net at C13.1, Q3.2 (B), R12.2: now also IC5.4 (RT/CT)
- net at R8.1: now also IC5.6 (OUT)
- net at R18.2: now also IC4.4 (COLLECTOR)
- net at R19.2: now also IC4.1 (ANODE)
- net at R22.2, R23.2: now also IC4.2 (CATHODE), IC6.3 (K)
- net at R14.1, R15.2: now also IC4.3 (EMMITER)
- new net: R13.2, R27.1
- no-connect marks 1 -> 0
Other:
- note added: "Añadir Ferrita a la alimentacion"
- note added: "Diseñar simbolo de MOV"
- note added: "Revisar Tierras. Probablemente la Tierra AC del flyback aislada. Y gnd salida DC = gnd alimentacion"
- note removed: "Anadir MOV y Capacitor de seguridad"
- moved on the sheet: R19

Commit message: Transformador-flyback-1
Parts:
- removed T2: Transformer_1P_2S, symbol Device:Transformer_1P_2S
- added T3: 750811351, 750811351, symbol F_1_750811351:750811351
Connections:
- net GNDREF: now also T3.7 (AUX_2)
- net at C16.1, C20.2, D5.1 (K)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: now also T3.2 (PRI_1)
- net at D12.2 (A), Q1.1 (D): now also T3.4 (PRI_3)
- net at R20.2: now also T3.6 (AUX_1)
- no-connect marks 0 -> 3
Other:
- moved on the sheet: C22, D13, J6

Commit message: Transformer-Connected
Connections:
- net GND: now also T3.10 (PRI_6), T3.8 (PRI_4), T3.9 (PRI_5)
- net at T3.12 (NC_4): now also D13.2 (A), T3.13 (PRI_7), T3.14 (PRI_8)
Other:
- moved on the sheet: C22, D13, J6

Commit message: Schematic-1-Flyback + 60HZ
Parts:
- removed R20, R8: R_Variable_US, symbol Device:R_Variable_US
- removed R6: R_US, symbol Device:R_US
- added FB1: FerriteBead, Flyback:BEADC1608X95N, symbol Device:FerriteBead
- added R28: 15, Resistor_SMD:R_1206_3216Metric_Pad1.30x1.75mm_HandSolder, symbol Device:R_US
- added R29: 22, Resistor_SMD:R_1206_3216Metric_Pad1.30x1.75mm_HandSolder, symbol Device:R_US
- C18: footprint (none) -> Capacitor_THT:CP_Radial_Tantal_D6.0mm_P2.50mm
- F1: footprint (none) -> Fuse:Fuseholder_Cylinder-5x20mm_Schurter_0031_8201_Horizontal_Open
- IC6: footprint TL431ACLPR -> Flyback:TL431ACLPR
- R14, R5: footprint (none) -> Resistor_SMD:R_0603_1608Metric_Pad0.98x0.95mm_HandSolder
- R16: value R_US -> 100; footprint (none) -> Resistor_SMD:R_1206_3216Metric_Pad1.30x1.75mm_HandSolder
- R17: value R_US -> 47k; footprint (none) -> Resistor_SMD:R_0603_1608Metric_Pad0.98x0.95mm_HandSolder
- R18: value R_Variable_US -> 200k; footprint (none) -> Potentiometer_THT:Potentiometer_Bourns_3296W_Vertical
- R21: footprint (none) -> Flyback:RESC6432X70N
- R26: value R_Variable_US -> 20k; footprint (none) -> Potentiometer_THT:Potentiometer_Bourns_3296W_Vertical
- RV1: footprint (none) -> Varistor:RV_Disc_D15.5mm_W4.4mm_P7.5mm
- T3: footprint 750811351 -> Flyback:750811351
Connections:
- net at D11.2 (A): now also R29.1
- net at T3.6 (AUX_1): now also R29.2
- net at C18.1, D11.1 (K), IC5.7 (VDD)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: now also FB1.1; no longer C19.2, D10.1 (K)
- net at IC5.6 (OUT): now also R28.1
- net at Q1.2 (G), R10.1: now also R28.2
- new net: C19.2, D10.1 (K), FB1.2
Other:
- note removed: "Añadir Ferrita a la alimentacion"
- note removed: "Diseñar simbolo de MOV"
- moved on the sheet: C19, D10

Commit message: PSIM-FLYBACK-FINAL
Parts:
- removed C21, C22: C, symbol Device:C
- removed R15: R_US, symbol Device:R_US
- added C22: 1000uF, Capacitor_THT:CP_Radial_D10.0mm_P5.00mm, symbol Device:C_Polarized
- added C24: 4.7uF, Capacitor_THT:CP_Radial_D10.0mm_P5.00mm, symbol Device:C_Polarized
- added C25: 10n, Capacitor_SMD:C_0805_2012Metric_Pad1.18x1.45mm_HandSolder, symbol Device:C
- added R20: 30k, Resistor_SMD:R_0603_1608Metric_Pad0.98x0.95mm_HandSolder, symbol Device:R_US
- added R30: 3k, Resistor_SMD:R_0603_1608Metric_Pad0.98x0.95mm_HandSolder, symbol Device:R_US
- C12: value 7n -> 10n
- C14: value C -> 3.3nF
- C16: value 618uF -> 680uF
- R19: value R_US -> 470k; footprint (none) -> Resistor_SMD:R_0603_1608Metric_Pad0.98x0.95mm_HandSolder
- R22: value R_US -> 470; footprint (none) -> Resistor_SMD:R_1206_3216Metric_Pad1.30x1.75mm_HandSolder
- R23: value R_US -> 24k; footprint (none) -> Resistor_SMD:R_0603_1608Metric_Pad0.98x0.95mm_HandSolder
- R24: value R_US -> 5.1k; footprint (none) -> Resistor_SMD:R_0603_1608Metric_Pad0.98x0.95mm_HandSolder
- R25: value R_US -> 1k; footprint (none) -> Resistor_SMD:R_0603_1608Metric_Pad0.98x0.95mm_HandSolder
Connections:
- net GND: now also R24.2, T3.12 (NC_4), T3.13 (PRI_7), T3.14 (PRI_8), C22.2, C24.2; no longer R25.2, T3.10 (PRI_6), T3.8 (PRI_4), T3.9 (PRI_5)
- net GNDREF: now also T3.6 (AUX_1); no longer T3.7 (AUX_2)
- net at R29.2: now also T3.7 (AUX_2); no longer T3.6 (AUX_1)
- net at R23.1: now also R25.2
- net at D13.1 (K), J6.1 (Pin_1), R19.1: now also R22.2, C22.1, C24.1, R20.1; no longer R22.1, R24.1
- net at C14.2, IC5.2 (FB), R7.2: now also R30.1
- net at IC4.2 (CATHODE), IC6.3 (K), R23.2: now also R22.1; no longer R22.2
- net at IC4.3 (EMMITER), R14.1: now also R30.2
- new net: D13.2 (A), T3.10 (PRI_6), T3.8 (PRI_4), T3.9 (PRI_5)
- new net: C25.1, IC6.1 (REF), R20.2, R24.1
- new net: C25.2, R25.1
Other:
- moved on the sheet: D13, J6

Commit message: Flyback-Routing1
Parts:
- removed D11, D12, D13: D_Filled, symbol Device:D_Filled
- removed D5, D6, D7, D8: 1N4007, Diode_THT:D_DO-41_SOD81_P10.16mm_Horizontal, symbol Diode:1N4007
- removed J6: Conn_01x02, Connector_JST:JST_XH_B2B-XH-A_1x02_P2.50mm_Vertical, symbol Connector_Generic:Conn_01x02
- removed Q1: NMOS, symbol Simulation_SPICE:NMOS
- removed Q2: PNP, symbol Simulation_SPICE:PNP
- removed Q3: NPN, symbol Simulation_SPICE:NPN
- added BR1: KBPC610, Flyback:KBPC610, symbol F_1_KBPC610:KBPC610
- added D14, D15, D16: ES3JB-HF, Flyback:DIOM5235X244N, symbol F_1_ES3JB-HF:ES3JB-HF
- added J5: TB002-500-02BE, Flyback:TB002-500-02BE, symbol F_1_TB002-500-02BE:TB002-500-02BE
- added Q1: BFR182E6327HTSA1, Flyback:NPN_SOT95P240X110-3N, symbol F_1_BFR182E6327HTSA1:BFR182E6327HTSA1
- added Q3: 2N3906BU, Flyback:2N3906BU, symbol F_1_2N3906BU:2N3906BU
- added Q4: Q_NMOS_GDS, Package_TO_SOT_THT:TO-220F-3_Vertical, symbol Transistor_FET:Q_NMOS_GDS
- C20: value C -> 1n; footprint (none) -> Capacitor_THT:C_Disc_D7.5mm_W4.4mm_P5.00mm
- C22: value 1000uF -> 680uF
- D10: value D_Zener_Filled -> +18; footprint (none) -> Diode_THT:D_DO-41_SOD81_P10.16mm_Horizontal
- D9: footprint (none) -> Diode_SMD:D_SMA_Handsoldering
- R19, R24: footprint Resistor_SMD:R_0603_1608Metric_Pad0.98x0.95mm_HandSolder -> Resistor_SMD:R_1206_3216Metric_Pad1.30x1.75mm_HandSolder
- R20: footprint Resistor_SMD:R_0603_1608Metric_Pad0.98x0.95mm_HandSolder -> Resistor_THT:R_Axial_DIN0414_L11.9mm_D4.5mm_P15.24mm_Horizontal
- R22: value 470 -> 100k; footprint Resistor_SMD:R_1206_3216Metric_Pad1.30x1.75mm_HandSolder -> Resistor_THT:R_Axial_DIN0414_L11.9mm_D4.5mm_P15.24mm_Horizontal
- R29: value 22 -> 100; footprint Resistor_SMD:R_1206_3216Metric_Pad1.30x1.75mm_HandSolder -> Resistor_THT:R_Axial_DIN0414_L11.9mm_D4.5mm_P15.24mm_Horizontal
- R9: value R_US -> 50k; footprint (none) -> Resistor_THT:R_Axial_Power_L50.0mm_W9.0mm_P60.96mm
Connections:
- net GND: now also J5.1
- net GNDREF: now also BR1.3 (-), Q3.3 (C)
- net Supplies/L: now also RV1.2, BR1.4 (~_2)
- net Supplies/N: now also F1.1; no longer RV1.2
- net Vref: now also Q1.3 (C)
- net at T3.10 (PRI_6), T3.8 (PRI_4), T3.9 (PRI_5): now also D15.2 (A)
- net at C16.1, C20.2, R5.1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: now also BR1.1 (+)
- net at T3.4 (PRI_3): now also D14.2 (A), Q4.2 (D)
- net at C22.1, C24.1, R19.1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: now also D15.1 (K), J5.2
- net at C11.2, D9.2 (A), R11.1: now also Q3.2 (B)
- net at C14.1, IC5.1 (COMP), R7.1: now also Q3.1 (E)
- net at F1.2: now also RV1.1, BR1.2 (~_1)
- net at C20.1, R9.1: now also D14.1 (K)
- net at C13.1, IC5.4 (RT/CT), R12.2: now also Q1.1 (B)
- net at C18.1, FB1.1, IC5.7 (VDD)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: now also D16.1 (K)
- net at C12.1: now also Q1.2 (E)
- net at R10.1, R28.2: now also Q4.1 (G)
- net at R29.1: now also D16.2 (A)
- net at R16.2, R21.1: now also Q4.3 (S)
- no-connect marks 3 -> 6
Other:
- note added: "Este RC si debe soportar altos voltajes. Aprox 1kV R9 disipa aprox: 0.5 a 1 W"
- note added: "Las resistencias 0603 soportan: 0.1W de disipacion. 75V max de nominal. 150V de trasientes cortos. Resistencias que no pueden ser 0603: R19 R22 R20 R29 R9"
- note added: "Las resistencias 1206 soportan (R < 1k): 0.25W de disipacion. 200V max de nominal. 400 V de trasientes cortos."
- note added: "Las resistencias ceramicas de 10W pueden tener: 10W. 1kV max nominal. Resistencias axiales normales de 1W: 1W 350V max nominal."
- note added: "R29 disipa bastante :/."
- moved on the sheet: C11, C20, C23, F1, J1, R29, R9, RV1

Commit message: Flyback-PCB-Final1
Parts:
- added FB5: FerriteBead, Flyback:BEADC1608X95N, symbol Device:FerriteBead
Connections:
- net GND: now also J5.2; no longer J5.1
- net at C22.1, C24.1, D15.1 (K)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: now also J5.1; no longer J5.2
- net at C18.1, D16.1 (K), FB1.1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: now also FB5.1; no longer R5.2
- new net: FB5.2, R5.2
Other:
- moved on the sheet: C18, D16, R29
