File: Electronic-design/General-Design/PCB/03_Power-supply-Flyback/Flyback_PCB_60Hz/PowerSupplies.kicad_sch (KiCad schematic)
At the start: 26 parts, among them IC1 TPS54302DDCR, IC2 L7812CV, IC3 L7912CV, J2 -12V, J3 +12V, J4 +5V, T1 3FS-324

Commit message: Wololo-Footprints-Flyback-1
Connections:
- net GNDREF renamed GND

Commit message: Schematic-1-Flyback + 60HZ
Parts:
- IC1: footprint SOT95P280X110-6N -> Footprints_Proyecto:SOT95P280X110-6N
- R2, R3: footprint R_0603_1608Metric_Pad0.98x0.95mm_HandSolder -> Resistor_SMD:R_0603_1608Metric_Pad0.98x0.95mm_HandSolder
Changed lines of the file:
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@@
 			)
 		)
-		(property "Footprint" "R_0603_1608Metric_Pad0.98x0.95mm_HandSolder"
+		(property "Footprint" "Resistor_SMD:R_0603_1608Metric_Pad0.98x0.95mm_HandSolder"
 			(at 221.996 127.254 90)
 			(effects
@@
 			)
 		)
-		(property "Footprint" "SOT95P280X110-6N"
+		(property "Footprint" "Footprints_Proyecto:SOT95P280X110-6N"
 			(at 201.93 182.55 0)
 			(effects
@@
 				)
 				(justify left top)
-				(hide yes)
 			)
 		)
@@
 			)
 		)
-		(property "Footprint" "R_0603_1608Metric_Pad0.98x0.95mm_HandSolder"
+		(property "Footprint" "Resistor_SMD:R_0603_1608Metric_Pad0.98x0.95mm_HandSolder"
 			(at 221.996 136.144 90)
 			(effects

Commit message: PSIM-FLYBACK-FINAL
Parts:
- added FB2, FB3, FB4: FerriteBead, Flyback:BEADC1608X95N, symbol Device:FerriteBead
Connections:
- net at C7.2, IC2.3 (OUTPUT): now also FB2.1; no longer J3.1 (Pin_1)
- net at C8.1, IC3.3 (OUT): now also FB3.1; no longer J2.1 (Pin_1)
- net at C3.1, C4.1, L1.2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: now also FB4.1; no longer J4.1 (Pin_1)
- new net: FB2.2, J3.1 (Pin_1)
- new net: FB3.2, J2.1 (Pin_1)
- new net: FB4.2, J4.1 (Pin_1)
Other:
- moved on the sheet: C3, C4, C5, IC1, J2, J3, J4, L1, R1, R2, R3

Commit message: Flyback-Routing1
Parts:
- C7, C8: value 100nF -> 220nF
Connections:
- no-connect marks 0 -> 1
Changed lines of the file:
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@@
 		(color 0 0 0 0)
+	)
+	(no_connect
+		(at 233.68 90.17)
 	)
 	(wire
@@
 			)
 		)
-		(property "Value" "100nF"
+		(property "Value" "220nF"
 			(at 133.096 91.948 0)
 			(effects
@@
 			)
 		)
-		(property "Value" "100nF"
+		(property "Value" "220nF"
 			(at 133.858 86.614 0)
 			(effects
